Commit message: Rviz fixes

File: project2/src/otherNodes/models/robots/pioneer.urdf (robot description, URDF)
Before this commit: robot pioneer3at_body, 18 links, 17 joints
Links:
- link chassis: geometry collision mesh filename=file:///workspaces/project2/src/otherNodes/models/meshes/ch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; visual mesh filename=file:///workspaces/project2/src/otherNodes/models/meshes/ch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
- link laser_frame: geometry collision box size=0.01 0.01 0.01; visual mesh filename=file:///workspaces/project2/src/otherNodes/models/meshes/ho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
- link p3at_back_left_axle: geometry collision box size=0.01 0.01 0.01; visual mesh filename=file:///workspaces/project2/src/otherNodes/models/meshes/p3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
- link p3at_back_left_hub: geometry collision box size=0.01 0.01 0.01; visual mesh filename=file:///workspaces/project2/src/otherNodes/models/meshes/p3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
- link p3at_back_left_wheel: geometry collision mesh filename=file:///workspaces/project2/src/otherNodes/models/meshes/p3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; visual mesh filename=file:///workspaces/project2/src/otherNodes/models/meshes/p3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
- link p3at_back_right_axle: geometry collision box size=0.01 0.01 0.01; visual mesh filename=file:///workspaces/project2/src/otherNodes/models/meshes/p3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
- link p3at_back_right_hub: geometry collision box size=0.01 0.01 0.01; visual mesh filename=file:///workspaces/project2/src/otherNodes/models/meshes/p3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
- link p3at_back_right_wheel: geometry collision mesh filename=file:///workspaces/project2/src/otherNodes/models/meshes/p3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; visual mesh filename=file:///workspaces/project2/src/otherNodes/models/meshes/p3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
- link p3at_front_left_axle: geometry collision box size=0.01 0.01 0.01; visual mesh filename=file:///workspaces/project2/src/otherNodes/models/meshes/p3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
- link p3at_front_left_hub: geometry collision box size=0.01 0.01 0.01; visual mesh filename=file:///workspaces/project2/src/otherNodes/models/meshes/p3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
- link p3at_front_left_wheel: geometry collision mesh filename=file:///workspaces/project2/src/otherNodes/models/meshes/p3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; visual mesh filename=file:///workspaces/project2/src/otherNodes/models/meshes/p3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
- link p3at_front_right_axle: geometry collision box size=0.01 0.01 0.01; visual mesh filename=file:///workspaces/project2/src/otherNodes/models/meshes/p3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
- link p3at_front_right_hub: geometry collision box size=0.01 0.01 0.01; visual mesh filename=file:///workspaces/project2/src/otherNodes/models/meshes/p3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
- link p3at_front_right_wheel: geometry collision mesh filename=file:///workspaces/project2/src/otherNodes/models/meshes/p3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; visual mesh filename=file:///workspaces/project2/src/otherNodes/models/meshes/p3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
- link top_plate: geometry collision box size=0.1 0.1 0.1; visual mesh filename=file:///workspaces/project2/src/otherNodes/models/meshes/to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

Commit message: Additions

File: project2/src/otherNodes/models/robots/pioneer.urdf (robot description, URDF)
Before this commit: robot pioneer3at_body, 18 links, 17 joints
Links:
- removed link laser_frame
- added link cloud, mass 1e-5; collision box size=0.01 0.01 0.01; visual mesh filename=file:///workspaces/project2/src/otherNodes/models/meshes/ho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
Joints:
- joint laser_joint: child laser_frame -> cloud

Commit message: Add stuff

File: project2/src/otherNodes/models/robots/pioneer.urdf (robot description, URDF)
Before this commit: robot pioneer3at_body, 18 links, 17 joints
Links:
- added link imu_link
Joints:
- added joint imu_joint: type fixed, parent base_link, child imu_link, origin xyz=0.3 0 0.2 rpy=0 0 0

Commit message: committ

File: project2/src/otherNodes/models/robots/pioneer.urdf (robot description, URDF)
Before this commit: robot pioneer3at_body, 19 links, 18 joints
Links:
- added link base_footprint
Joints:
- added joint base_link_to_footprint: type fixed, parent base_link, child base_footprint, origin xyz=0 0 0 rpy=0 0 0
- joint imu_joint: parent base_link -> base_footprint
- joint laser_joint: parent chassis -> base_footprint

Commit message: Update pioneer.urdf
pion

File: project2/src/otherNodes/models/robots/pioneer.urdf (robot description, URDF)
Before this commit: robot pioneer3at_body, 20 links, 19 joints
Links:
- removed link cam_optical_link
- added link oak-d-base-frame
Joints:
- joint cam_optical_joint: child cam_optical_link -> oak-d-base-frame
